Commit message: Modified urdf
Signed-off-by: Pyo <pyo@robotis.com>

File: testbot_description/urdf/testbot.urdf (robot description, URDF)
Before this commit: robot testbot, 5 links, 4 joints
Links:
- link link1: mass 1 -> 1.0
- link link2: mass 1 -> 1.0
- link link3: mass 1 -> 1.0; geometry collision box size=0.1 0.1 1.0; visual box size=0.1 0.1 1.0
- link link4: mass 1 -> 1.0
Joints:
- joint joint1: axis 0 0 1 -> 0.0 0.0 1.0; limit lower=-2.617 upper=2.617 effort=30 velocity=1.571 -> lower=-2.617 upper=2.617 effort=30.0 velocity=1.571; origin xyz=0 0 0.5 rpy=0 0 0 -> xyz=0.0 0.0 0.5 rpy=0.0 0.0 0.0
- joint joint2: axis 0 1 0 -> 0.0 1.0 0.0; limit lower=-2.617 upper=2.617 effort=30 velocity=1.571 -> lower=-2.617 upper=2.617 effort=30.0 velocity=1.571; origin xyz=0 0 0.5 rpy=0 0 0 -> xyz=0.0 0.0 0.5 rpy=0.0 0.0 0.0
- joint joint3: axis 0 1 0 -> 0.0 1.0 0.0; limit lower=-2.617 upper=2.617 effort=30 velocity=1.571 -> lower=-2.617 upper=2.617 effort=30.0 velocity=1.571; origin xyz=0 0 1.0 rpy=0 0 0 -> xyz=0.0 0.0 1.0 rpy=0.0 0.0 0.0
